File: Entrenador PIC18F4550/PIC18F4550/PIC18F4550.kicad_pcb (KiCad board)
At the start: 2 copper layers, 70 x 88 mm, 32 parts, among them J1 Barrel_Jack_Switch, J10 PORTA, J11 PORTC, J12 UART_TTL, J2 Alimenatciones, J3 PICKIT, J5 Conn_01x03_Male, J6 USB_B, J7 PORTE, J8 PORTB, J9 PORTD, SW1 RESET, U1 KA378R33, U2 L7805, U3 PIC18F4550-IP, Y1 Crystal

Commit message: Pcbs
Parts:
- moved C2 25.9 mm to (139.6, 146.4)
- moved C5 7.64 mm to (125.2, 132.0), turned to 90 degrees
- moved C4 2.31 mm to (133.2, 145.2)
- moved C3 0.21 mm to (132.8, 155.4)
Routing:
- net GND: track 331.4 -> 0.00 mm, vias 14 -> 0
- net 5V: track 212.3 -> 0.00 mm, vias 8 -> 0
- net /RC4: track 91.9 -> 0.00 mm, vias 6 -> 0
- net /RC5: track 86.7 -> 0.00 mm, vias 6 -> 0
- net /RC7: track 83.8 -> 0.00 mm, vias 6 -> 0
- net /RC6: track 78.3 -> 0.00 mm, vias 2 -> 0
- net 3.3V: track 64.0 -> 0.00 mm, vias 4 -> 0
- net /RB6: track 59.8 -> 0.00 mm
- net /RB7: track 57.8 -> 0.00 mm
- net /RD0: track 47.3 -> 0.00 mm
- net Net-(JP2-Pad2): track 40.9 -> 0.00 mm, vias 2 -> 0
- net /PUSH_RESET: track 40.1 -> 0.00 mm
- net /RD1: track 39.6 -> 0.00 mm
- net Net-(C3-Pad1): track 36.4 -> 0.00 mm
- net /RC2: track 32.6 -> 0.00 mm
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- removed copper zone on B.Cu, net GND
