File: Inyectores_JLCPCB/Principal/CIRCUITO.sch (KiCad schematic (older format))
At the start: 28 parts, among them J2 Screw_Terminal_01x03, J3 Screw_Terminal_01x02, U2 PIC16F886-IP, U7 LM35-LP, Y1 20MHz

Commit message: -
Parts:
- removed J3: Screw_Terminal_01x02, Connector_PinSocket_2.54mm:PinSocket_1x02_P2.54mm_Vertical, symbol Connector:Screw_Terminal_01x02
- removed POTE_IN1: Screw_Terminal_01x05, Connector_PinHeader_2.54mm:PinHeader_1x05_P2.54mm_Vertical, symbol Connector:Screw_Terminal_01x05
- removed PULSADORES_IN1: Screw_Terminal_01x07, Connector_PinHeader_2.54mm:PinHeader_1x07_P2.54mm_Vertical, symbol Connector:Screw_Terminal_01x07
- POTE_OUT1: footprint Connector_PinHeader_2.54mm:PinHeader_1x05_P2.54mm_Vertical -> Connector_PinSocket_2.54mm:PinSocket_1x05_P2.54mm_Vertical
- PULSADORES_OUT1: footprint Connector_PinHeader_2.54mm:PinHeader_1x07_P2.54mm_Vertical -> Connector_PinSocket_2.54mm:PinSocket_1x07_P2.54mm_Vertical
Connections:
- net GND_POTE is gone; now on net GND: MIN1.3, PWM1.3, RPM1.3
- net GND_PULS is gone; now on net GND: DET_10K1.2, DRE_10K1.2, ENT_10K1.2, MOV_10K1.2, RESET1.1
- net VCC_POTE is gone; now on net 5V: MIN1.1, PWM1.1, RPM1.1
- net VCC_PULS is gone; now on net 5V: DETENER1.2, DRENAJE1.2, ENTER1.2, MOVER1.2, RES_10K1.2
- net DETENER: now also PULSADORES_OUT1.3 (Pin_3), U2.23 (P1B/AN8/RB2)
- net DRENAJE: now also PULSADORES_OUT1.1 (Pin_1), U2.21 (INT/AN12/RB0)
- net ENTER: now also PULSADORES_OUT1.2 (Pin_2), U2.22 (P1C/AN10/RB1)
- net MCLR: now also J2.1 (Pin_1), PULSADORES_OUT1.5 (Pin_5)
- net MIN: now also POTE_OUT1.3 (Pin_3), U2.4 (CVref/C2IN1+/Vref-/AN2/RA2)
- net MOVER: now also PULSADORES_OUT1.4 (Pin_4), U2.24 (PGM/C12IN2-/AN8/RB3)
- net OUT: now also U2.13 (RC2/P1A/CCP1); no longer U2.25 (P1D/AN11/RB4)
- net PWM: now also POTE_OUT1.2 (Pin_2), U2.3 (C12IN1-/AN1/RA1)
- net RPM: now also POTE_OUT1.1 (Pin_1), U2.2 (ULPWU/C12IN0-/AN0/RA0)
- net RB4: now reaches LCD_OUT1.8 (Pin_8)
- net RB4: now also U2.25 (P1D/AN11/RB4); no longer U2.13 (RC2/P1A/CCP1)
- net Buzzer: now reaches BZ1.1 (-), U2.7 (~SS~/C2OUT/AN4/RA5)
- net RA4 renamed RELE1
- net RB5 renamed RELE2
Other:
- moved on the sheet: BZ1, C3, C4, DETENER1, DET_10K1, DRENAJE1, DRE_10K1, ENTER1, ENT_10K1, J2, LCD1, MIN1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
