File: Inyectores_JLCPCB/Principal/FUENTE.sch (KiCad schematic (older format))
At the start: 6 parts, among them J4 ENTRADA_CIRCUITO, U1 L7805

Commit message: -
Parts:
- J4: footprint BorneraTornillos:bornera_tornillos_1x03 -> BorneraTornillos:TerminalBlock_Phoenix_PT-1,5-3-5.0-H_1x03_P5.00mm_Horizontal
Connections:
- net GND: now also J4.1 (Pin_1); no longer J4.3 (Pin_3)
- net VCC: now also J4.3 (Pin_3); no longer J4.1 (Pin_1)
Changed lines of the file:
@@
 EESchema Schematic File Version 4
+LIBS:INYECTORES-cache
 EELAYER 30 0
 EELAYER END
@@
 U 1 1 5F38743A
 P 4500 3500
-F 0 "J4" H 4418 3817 50  0000 C CNN
-F 1 "ENTRADA_CIRCUITO" H 4418 3726 50  0000 C CNN
-F 2 "BorneraTornillos:bornera_tornillos_1x03" H 4500 3500 50  0001 C CNN
+F 0 "J4" H 4450 3900 50  0000 C CNN
+F 1 "ENTRADA_CIRCUITO" H 4450 3800 50  0000 C CNN
+F 2 "BorneraTornillos:TerminalBlock_Phoenix_PT-1,5-3-5.0-H_1x03_P5.00mm_Horizontal" H 4500 3500 50  0001 C CNN
 F 3 "~" H 4500 3500 50  0001 C CNN
 	1    4500 3500
-	-1   0    0    -1
+	-1   0    0    1
 $EndComp
 Wire Wire Line
