File: Inyectores_JLCPCB/Principal/INYECTORES.kicad_pcb (KiCad board)
At the start: 2 copper layers, 100 x 100 mm, 58 parts, among them J2 Screw_Terminal_01x03, J3 Screw_Terminal_01x02, J4 ENTRADA_CIRCUITO, J5 INY2, J6 INY1, J7 INY4, J8 INY3, Q1 IRF540N, Q2 IRF540N, Q3 IRF540N, Q4 IRF540N, U1 L7805, U2 PIC16F886-IP, U3 PC817_INY1, U4 PC817_INY2, U5 PC817_INY3, U6 PC817_INY4, U7 LM35-LP, Y1 20MHz

Commit message: -
Parts:
- removed J8: INY3, BorneraTornillos:bornera_tornillos_1x03
- removed POTE_IN1: Screw_Terminal_01x05, Connector_PinHeader_2.54mm:PinHeader_1x05_P2.54mm_Vertical
- removed PULSADORES_IN1: Screw_Terminal_01x07, Connector_PinHeader_2.54mm:PinHeader_1x07_P2.54mm_Vertical
- added C5: 104, Capacitor_THT:C_Disc_D3.4mm_W2.1mm_P2.50mm, F.Cu at (142.5, 112.5)
- added C6: 104, Capacitor_THT:C_Disc_D3.4mm_W2.1mm_P2.50mm, F.Cu at (127.5, 112.5)
- added C7: 104, Capacitor_THT:C_Disc_D3.4mm_W2.1mm_P2.50mm, F.Cu at (137.0, 112.5)
- added C8: 104, Capacitor_THT:C_Disc_D3.4mm_W2.1mm_P2.50mm, F.Cu at (152.0, 112.5)
- added D10: LED, LED_SMD:LED_0805_2012Metric, F.Cu at (137.0, 96.0)
- added D11: Rele 2, LED_SMD:LED_0805_2012Metric, F.Cu at (147.5, 96.0)
- added D12: Rele 1, LED_SMD:LED_0805_2012Metric, F.Cu at (151.0, 96.0)
- added D13: 1N4007, Diode_THT:D_DO-41_SOD81_P10.16mm_Horizontal, F.Cu at (185.2, 113.3)
- added D14: 1N4007, Diode_THT:D_DO-41_SOD81_P10.16mm_Horizontal, F.Cu at (168.8, 113.2)
- added D7: LED, LED_SMD:LED_0805_2012Metric, F.Cu at (140.5, 96.0)
- added D8: LED, LED_SMD:LED_0805_2012Metric, F.Cu at (133.5, 96.0)
- added D9: LED, LED_SMD:LED_0805_2012Metric, F.Cu at (144.0, 96.0)
- added J1: INYECTORES, BorneraTornillos:TerminalBlock_Phoenix_PT-1,5-3-5.0-H_1x03_P5.00mm_Horizontal, F.Cu at (129.0, 141.0)
- added K1: SANYOU_SRD_Form_C, Relay_THT:Relay_SPDT_SANYOU_SRD_Series_Form_C, F.Cu at (180.0, 117.5)
- added K2: SANYOU_SRD_Form_C, Relay_THT:Relay_SPDT_SANYOU_SRD_Series_Form_C, F.Cu at (163.5, 117.5)
- added Q5: 2N2219, Package_TO_SOT_THT:TO-92_Inline, F.Cu at (173.6, 109.4)
- added Q6: 2N2219, Package_TO_SOT_THT:TO-92_Inline, F.Cu at (179.4, 109.4)
- added R1: 180, Resistor_THT:R_Axial_DIN0207_L6.3mm_D2.5mm_P10.16mm_Horizontal, F.Cu at (173.0, 97.0)
- added R11: 180, Resistor_THT:R_Axial_DIN0207_L6.3mm_D2.5mm_P10.16mm_Horizontal, F.Cu at (183.0, 104.0)
- added R12: 180, Resistor_THT:R_Axial_DIN0207_L6.3mm_D2.5mm_P10.16mm_Horizontal, F.Cu at (183.0, 100.5)
- added R2: 180, Resistor_THT:R_Axial_DIN0207_L6.3mm_D2.5mm_P10.16mm_Horizontal, F.Cu at (167.0, 97.0)
- added REF**: KiCad-Logo2_20mm_SilkScreen, Symbol:KiCad-Logo2_20mm_SilkScreen, B.Cu at (152.0, 72.0)
- added REF1: MountingHole_3.2mm_M3_Pad, MountingHole:MountingHole_3.2mm_M3_Pad, F.Cu at (105.0, 54.5)
- added REF2: MountingHole_3.2mm_M3_Pad, MountingHole:MountingHole_3.2mm_M3_Pad, F.Cu at (195.0, 54.5)
- added REF3: MountingHole_3.2mm_M3_Pad, MountingHole:MountingHole_3.2mm_M3_Pad, F.Cu at (105.0, 145.5)
- added REF4: MountingHole_3.2mm_M3_Pad, MountingHole:MountingHole_3.2mm_M3_Pad, F.Cu at (195.0, 145.5)
- added U8: PC817_INY2, Package_DIP:DIP-4_W7.62mm_LongPads, F.Cu at (167.4, 101.0)
- added U9: PC817_INY2, Package_DIP:DIP-4_W7.62mm_LongPads, F.Cu at (160.2, 101.1)
- J3: value Screw_Terminal_01x02 -> RELE1; footprint Connector_PinSocket_2.54mm:PinSocket_1x02_P2.54mm_Vertical -> BorneraTornillos:TerminalBlock_Phoenix_PT-1,5-3-5.0-H_1x03_P5.00mm_Horizontal
- J4: footprint BorneraTornillos:bornera_tornillos_1x03 -> BorneraTornillos:TerminalBlock_Phoenix_PT-1,5-3-5.0-H_1x03_P5.00mm_Horizontal
- J5: value INY2 -> INYECTORES; footprint BorneraTornillos:bornera_tornillos_1x03 -> BorneraTornillos:TerminalBlock_Phoenix_PT-1,5-2-5.0-H_1x02_P5.00mm_Horizontal
- J6: value INY1 -> INYECTORES; footprint BorneraTornillos:bornera_tornillos_1x03 -> BorneraTornillos:TerminalBlock_Phoenix_PT-1,5-3-5.0-H_1x03_P5.00mm_Horizontal
- J7: value INY4 -> RELE2; footprint BorneraTornillos:bornera_tornillos_1x03 -> BorneraTornillos:TerminalBlock_Phoenix_PT-1,5-3-5.0-H_1x03_P5.00mm_Horizontal
- POTE_OUT1: footprint Connector_PinHeader_2.54mm:PinHeader_1x05_P2.54mm_Vertical -> Connector_PinSocket_2.54mm:PinSocket_1x05_P2.54mm_Vertical
- PULSADORES_OUT1: footprint Connector_PinHeader_2.54mm:PinHeader_1x07_P2.54mm_Vertical -> Connector_PinSocket_2.54mm:PinSocket_1x07_P2.54mm_Vertical
- Q1, Q2, Q3, Q4: footprint Package_TO_SOT_THT:TO-220-3_Horizontal_TabDown -> Package_TO_SOT_THT:TO-220-3_Vertical
- moved D3 157.7 mm to (103.5, 118.1), turned to 270 degrees
- moved R5 155.4 mm to (112.5, 104.0), turned to 270 degrees
- moved D4 148.4 mm to (110.0, 118.1), turned to 270 degrees
- moved R8 132.8 mm to (123.0, 104.0), turned to 270 degrees
- moved R3 124.3 mm to (138.5, 120.5), turned to 180 degrees
- moved R4 118.8 mm to (138.5, 116.5), turned to 180 degrees
- moved D5 115.8 mm to (116.5, 118.1), turned to 270 degrees
- moved R9 112.9 mm to (152.5, 116.5), turned to 180 degrees
- moved R10 112.9 mm to (152.5, 120.5), turned to 180 degrees
- moved D6 106.5 mm to (123.0, 118.1), turned to 270 degrees
- moved DETENER1 99.3 mm to (108.0, 107.0), turned to 270 degrees
- moved R6 98.5 mm to (116.0, 104.0), turned to 270 degrees
- moved R7 97.4 mm to (119.5, 104.0), turned to 270 degrees
- moved DET_10K1 93.1 mm to (122.0, 99.0), turned to 90 degrees
- moved DRENAJE1 89.2 mm to (108.0, 97.0), turned to 270 degrees
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Connections:
- net Net-(BZ1-Pad1) renamed /CIRCUITO/Buzzer
- net Net-(D5-Pad2) renamed /SALIDA/COM_INY_3
- D3 pad 2: Net-(D3-Pad2) -> /SALIDA/COM_INY_1
- D4 pad 2: Net-(D4-Pad2) -> /SALIDA/COM_INY_2
- D6 pad 2: Net-(D6-Pad2) -> /SALIDA/COM_INY_4
- DETENER1 pad 2: /CIRCUITO/VCC_PULS -> 5V
- DET_10K1 pad 2: /CIRCUITO/GND_PULS -> GND
- DRENAJE1 pad 2: /CIRCUITO/VCC_PULS -> 5V
- DRE_10K1 pad 2: /CIRCUITO/GND_PULS -> GND
- ENTER1 pad 2: /CIRCUITO/VCC_PULS -> 5V
- ENT_10K1 pad 2: /CIRCUITO/GND_PULS -> GND
- J2 pad 1: Net-(J2-Pad1) -> /CIRCUITO/MCLR
- J3 pad 1: /CIRCUITO/RA4 -> /SALIDA/RELE1_NA
- J3 pad 2: /CIRCUITO/RB5 -> /SALIDA/COM_RELE1
- J4 pad 1: 12V -> GND
- J4 pad 3: GND -> 12V
- J5 pad 2: Net-(J5-Pad2) -> /SALIDA/COM_INY_4
- J6 pad 2: Net-(J6-Pad2) -> /SALIDA/COM_INY_1
- J6 pad 3: Net-(D3-Pad2) -> 12V
- J7 pad 1: 12V -> /SALIDA/RELE2_NA
- J7 pad 2: Net-(J7-Pad2) -> /SALIDA/COM_RELE2
- J7 pad 3: Net-(D6-Pad2) -> /SALIDA/RELE2_NC
- LCD_OUT1 pad 8: Net-(LCD_OUT1-Pad8) -> /CIRCUITO/RB4
- MIN1 pad 1: /CIRCUITO/VCC_POTE -> 5V
- MIN1 pad 3: /CIRCUITO/GND_POTE -> GND
- MOVER1 pad 2: /CIRCUITO/VCC_PULS -> 5V
- MOV_10K1 pad 2: /CIRCUITO/GND_PULS -> GND
- POTE_OUT1 pad 1: Net-(POTE_OUT1-Pad1) -> /CIRCUITO/RPM
- POTE_OUT1 pad 2: Net-(POTE_OUT1-Pad2) -> /CIRCUITO/PWM
- POTE_OUT1 pad 3: Net-(POTE_OUT1-Pad3) -> /CIRCUITO/MIN
- PULSADORES_OUT1 pad 1: Net-(PULSADORES_OUT1-Pad1) -> /CIRCUITO/DRENAJE
- PULSADORES_OUT1 pad 2: Net-(PULSADORES_OUT1-Pad2) -> /CIRCUITO/ENTER
- PULSADORES_OUT1 pad 3: Net-(PULSADORES_OUT1-Pad3) -> /CIRCUITO/DETENER
- PULSADORES_OUT1 pad 4: Net-(PULSADORES_OUT1-Pad4) -> /CIRCUITO/MOVER
- PULSADORES_OUT1 pad 5: Net-(J2-Pad1) -> /CIRCUITO/MCLR
- PWM1 pad 1: /CIRCUITO/VCC_POTE -> 5V
- PWM1 pad 3: /CIRCUITO/GND_POTE -> GND
- Q1 pad 2: Net-(D3-Pad2) -> /SALIDA/COM_INY_1
- Q2 pad 2: Net-(D4-Pad2) -> /SALIDA/COM_INY_2
- Q4 pad 2: Net-(D6-Pad2) -> /SALIDA/COM_INY_4
- RESET1 pad 1: /CIRCUITO/GND_PULS -> GND
- RES_10K1 pad 2: /CIRCUITO/VCC_PULS -> 5V
- RPM1 pad 1: /CIRCUITO/VCC_POTE -> 5V
- RPM1 pad 3: /CIRCUITO/GND_POTE -> GND
- U2 pad 13: Net-(LCD_OUT1-Pad8) -> OUT
- U2 pad 2: Net-(POTE_OUT1-Pad1) -> /CIRCUITO/RPM
- U2 pad 21: Net-(PULSADORES_OUT1-Pad1) -> /CIRCUITO/DRENAJE
- U2 pad 22: Net-(PULSADORES_OUT1-Pad2) -> /CIRCUITO/ENTER
- U2 pad 23: Net-(PULSADORES_OUT1-Pad3) -> /CIRCUITO/DETENER
- U2 pad 24: Net-(PULSADORES_OUT1-Pad4) -> /CIRCUITO/MOVER
- U2 pad 25: OUT -> /CIRCUITO/RB4
- U2 pad 26: /CIRCUITO/RB5 -> RELE2
- U2 pad 3: Net-(POTE_OUT1-Pad2) -> /CIRCUITO/PWM
- U2 pad 4: Net-(POTE_OUT1-Pad3) -> /CIRCUITO/MIN
- U2 pad 6: /CIRCUITO/RA4 -> RELE1
- U3 pad 2: GND -> Net-(D8-Pad2)
- U3 pad 4: 12V -> 5V
- U4 pad 2: GND -> Net-(D10-Pad2)
- U4 pad 4: 12V -> 5V
- U5 pad 2: GND -> Net-(D7-Pad2)
- U5 pad 4: 12V -> 5V
- U6 pad 2: GND -> Net-(D9-Pad2)
- U6 pad 4: 12V -> 5V
Routing:
- net GND: track 0.00 -> 447.2 mm
- net 5V: track 0.00 -> 375.0 mm
- net 12V: track 0.00 -> 319.0 mm
- net /CIRCUITO/DETENER: track 0.00 -> 87.8 mm
- net /CIRCUITO/MOVER: track 0.00 -> 85.4 mm
- net /CIRCUITO/ENTER: track 0.00 -> 84.0 mm
- net OUT: track 0.00 -> 78.3 mm
- net /CIRCUITO/DRENAJE: track 0.00 -> 72.7 mm
- net /CIRCUITO/MCLR: track 0.00 -> 67.0 mm
- net /SALIDA/COM_INY_3: track 0.00 -> 63.3 mm
- net /SALIDA/COM_INY_2: track 0.00 -> 61.5 mm
- net Net-(LCD_OUT1-Pad4): track 0.00 -> 61.3 mm, vias 0 -> 1
- net /CIRCUITO/RPM: track 0.00 -> 60.0 mm
- net Net-(C8-Pad1): track 0.00 -> 58.6 mm
- net /CIRCUITO/ICSPDAT: track 0.00 -> 53.1 mm
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- added copper zone on B.Cu, net GND
- added copper zone on F.Cu, net GND
Other:
- outline, holes or cut-outs redrawn
- net class Default: trace_width 0.25 -> 0.3
- net class Pcb_Casera removed
- net class Potencia added: clearance 0.5, trace_width 2.5, via_dia 1.7, via_drill 0.5
- rule trace_min: 0.25 -> 0.3
- board text added: "COM_INY2 INY3 COM_INY3"
- board text added: "DETENER"
- board text added: "DRENAJE"
- board text added: "ENTER"
- board text added: "GND 12V"
- board text added: "INY1"
- board text added: "INY1 COM_INY1 INY2"
- board text added: "INY2"
- board text added: "INY3"
- board text added: "INY4"
- board text added: "INY4 COM_INY4"
- board text added: "MOVER"
- board text added: "NORM PROMG"
- board text added: "RELE1_NA COM_RELE1 RELE1_NC"
- board text added: "RELE1_ON"
- board text added: "RELE2_NA COM_RELE2 RELE2_NC"
- board text added: "RELE2_ON"
- board text added: "RESET"
