File: Placa_Desarrollo_RPI-pico/Alimentacion.sch (KiCad schematic (older format))
At the start: 15 parts, among them J1 Barrel_Jack_Switch, SW1 SW_Push_SPDT, U1 L7805, U2 LT1083-3.3

Commit message: -
Parts:
- removed U2: LT1083-3.3, symbol Regulator_Linear:LT1083-3.3
- added D16: LED POWER 12V, symbol Device:LED
- added R26: 185, symbol Device:R
- added U2: AMS1117-3.3, Package_TO_SOT_SMD:SOT-223-3_TabPin2, symbol Regulator_Linear:AMS1117-3.3
- D3: value LED -> LED POWER 5V
- D4: value LED -> LED POWER 3.3V
- JP1: value Jumper_3_Bridged12 -> JUMPER 5V
- R1: value R -> 185
- R2: value R -> 100
Connections:
- net +12V: now also R26.1
- net +3V3: now also U2.2 (VO)
- net +5V: now also U2.3 (VI)
- net GND: now also D16.1 (K), U2.1 (GND)
- net VUSB renamed VBUS
- new net: D16.2 (A), R26.2
Other:
- moved on the sheet: D1
