File: Placa_Desarrollo_RPI-pico/Conectividad.sch (KiCad schematic (older format))
At the start: 14 parts, among them J7 Conn_01x20_Female, J8 Conn_01x08_Female, Q5 BC548, U8 24LC256

Commit message: -
Parts:
- removed DS3231: Conn_01x06_Female, symbol Connector:Conn_01x06_Female
- removed J7: Conn_01x20_Female, symbol Connector:Conn_01x20_Female
- removed J8: Conn_01x08_Female, symbol Connector:Conn_01x08_Female
- removed Q5: BC548, Package_TO_SOT_THT:TO-92_Inline, symbol Placa_Desarrollo_RPI-pico-cache:BC548
- added J10: WIFI1, symbol Connector:Conn_01x04_Female
- added J11: WIFI2, symbol Connector:Conn_01x04_Female
- added J14: LCD_I2C, symbol Connector:Conn_01x04_Female
- added J6: DS3231, symbol Connector:Conn_01x10_Female
- added JP2, JP3, JP4: RST, symbol Device:Jumper
- added JP9: CH_PD, symbol Device:Jumper
- added R25, R3, R4, R5: 10K, symbol Device:R
- JP5: value Jumper_2_Open -> A0
- JP6: value Jumper_2_Open -> A1
- JP7: value Jumper_2_Open -> A2
Connections:
- net +5V is gone; now on net +3V3: Bluetooth1.1 (Pin_1), JP5.1 (A), JP6.1 (A), JP7.1 (A), JP8.2 (B), U8.8 (VCC)
- net +3V3: now also J10.4 (Pin_4), J14.2 (Pin_2), J6.2 (Pin_2), JP2.2, JP3.2, JP4.2, JP9.2
- net GND: now also J11.1 (Pin_1), J14.1 (Pin_1), J6.1 (Pin_1), R25.2, R3.2, R4.2, R5.2
- net SCL renamed SCL0
- net SCL0: now also J14.4 (Pin_4), J6.4 (Pin_4)
- net SDA renamed SDA0
- net SDA0: now also J14.3 (Pin_3), J6.3 (Pin_3)
- net Uart_Rx0 renamed RX0
- net RX0: now also J10.1 (Pin_1)
- net Uart_Tx0 renamed TX0
- net TX0: now also J11.4 (Pin_4)
- new net CH_PD: J10.2 (Pin_2), JP9.1, R25.1
- new net GPIO0: J11.3 (Pin_3), JP4.1, R5.1
- new net GPIO2: J11.2 (Pin_2), JP3.1, R4.1
- new net RST: J10.3 (Pin_3), JP2.1, R3.1
- no-connect marks 15 -> 6
Other:
- moved on the sheet: Bluetooth1, JP5, JP6, JP7
