File: Placa_Desarrollo_RPI-pico/Micro.sch (KiCad schematic (older format))
At the start: 8 parts, among them J13 Conn_01x02_Female, Q14 BC548, U10 PICO_RP2040

Commit message: -
Parts:
- removed JP12, JP13: Jumper_3_Bridged12, symbol Jumper:Jumper_3_Bridged12
- removed Q14: BC548, Package_TO_SOT_THT:TO-92_Inline, symbol Placa_Desarrollo_RPI-pico-cache:BC548
- added D14: 1N5819, Diode_THT:D_DO-41_SOD81_P10.16mm_Horizontal, symbol Diode:1N5819
- added J15: Conn_01x07_Female, symbol Connector:Conn_01x07_Female
- added JP10: 5V RPI PICO, symbol Device:Jumper
- added SW6: RESET, symbol Switch:SW_Push
- J13: value Conn_01x02_Female -> PINES_PIO
- R34, R35: value R -> 2K2
Connections:
- net PUSH1 is gone; now on net A_ENC: U10.9 (GP6)
- net PUSH2 is gone; now on net B_ENC: U10.10 (GP7)
- net +3V3: now also J15.1 (Pin_1)
- net +5V: now also D14.2 (A); no longer BZ1.1 (-)
- net A_ENC: no longer U10.12 (GP9)
- net B_ENC: no longer U10.14 (GP10)
- net GND: now also BZ1.2 (+), J15.2 (Pin_2), SW6.1
- net GP15: now also J15.4 (Pin_4)
- net GP18: now also J15.5 (Pin_5)
- net GP19: now also J15.6 (Pin_6)
- net GP22: now also J15.7 (Pin_7)
- net Reset: now also SW6.2
- net at U10.39 (VSYS): now also JP10.1
- net VBUS: now reaches U10.40 (VBUS)
- net BRILLO_PWM renamed GP14
- net GP14: now also J15.3 (Pin_3)
- net GP0 renamed TX0
- net GP1 renamed RX0
- net Motor_1 renamed TOUCH3
- net Motor_2 renamed BUZZER
- net BUZZER: now also BZ1.1 (-)
- net PIO1 renamed GP16
- net GP16: now also U10.21 (GP16); no longer U10.22 (GP17)
- net PIO2 renamed GP17
- net GP17: now also U10.22 (GP17); no longer U10.21 (GP16)
- net SCL renamed SCL0
- net SDA renamed SDA0
- net SPI0_CS0 renamed MOSFET2
- net SPI0_CS1 renamed RELE_SS
- net SPI0_SDI renamed RELE2
- net SPI0_SDO renamed MOSFET1
- net SPI0_SLCK renamed RELE1
- new net: D14.1 (K), JP10.2
- new net TOUCH1: U10.12 (GP9)
- new net TOUCH2: U10.14 (GP10)
- no-connect marks 7 -> 3
Other:
- note added: "Conectividad"
- note added: "Pines"
- note added: "RASPBERRY PI PICO"
- note added: "Reset"
- moved on the sheet: BZ1, J13, R34, R35, U10
