File: Placa_Desarrollo_RPI-pico/Salida_Motor.sch (KiCad schematic (older format))
At the start: 22 parts, among them J12 Screw_Terminal_01x02, Q10 BC548, Q11 IRF540NPBF, Q12 IRF540NPBF, Q13 BC548, Q6 BC548, Q7 IRF540NPBF, Q8 IRF540NPBF, Q9 BC548, U9 LM358

Commit message: -
Parts:
- removed D16, D17: 1N4007, Diode_THT:D_DO-41_SOD81_P10.16mm_Horizontal, symbol Diode:1N4007
- removed Q10, Q13, Q6, Q9: BC548, Package_TO_SOT_THT:TO-92_Inline, symbol Placa_Desarrollo_RPI-pico-cache:BC548
- removed Q12, Q8: IRF540NPBF, digikey-footprints:TO-220-3, symbol Placa_Desarrollo_RPI-pico-rescue:IRF540NPBF-dk_Transistors-FETs-MOSFETs-Single
- removed R26, R28, R29, R30, R32, R33: R, symbol Device:R
- removed U9: LM358, symbol Amplifier_Operational:LM358
- added J5: Terminal M2, symbol Connector:Screw_Terminal_01x02
- J12: value Screw_Terminal_01x02 -> Terminal M1
Connections:
- net +12V: now also D18.1 (K), J12.1 (Pin_1), J5.1 (Pin_1); no longer Q7.2 (D)
- net GND: now also Q7.3 (S); no longer D18.2 (A)
- net COM_MOSFET1: now reaches J12.2 (Pin_2)
- net COM_MOSFET1: now also D15.2 (A), Q7.2 (D)
- net Mosfet_1 renamed MOSFET1
- net Mosfet_3 renamed MOSFET2
- new net COM_MOSFET2: D18.2 (A), J5.2 (Pin_2), Q11.2 (D)
Other:
- moved on the sheet: D15, D18, J12, Q11, Q7, R27, R31
