File: Placa_Desarrollo_RPI-pico/Salida_Potencia.sch (KiCad schematic (older format))
At the start: 38 parts, among them J2 Screw_Terminal_01x03, J3 Screw_Terminal_01x03, J4 Screw_Terminal_01x03, J5 Screw_Terminal_01x02, J6 Screw_Terminal_01x02, K1 DIPxx-1Cxx-51x, K2 DIPxx-1Cxx-51x, K3 DIPxx-1Cxx-51x, Q1 BC548, Q2 BC548, Q3 BC548, Q4 BT138-800, U3 PCF8574, U4 PC817, U5 PC817, U6 PC817, U7 MOC3021M

Commit message: -
Parts:
- removed D10: LED, symbol Device:LED
- removed D7: 1N4007, Diode_THT:D_DO-41_SOD81_P10.16mm_Horizontal, symbol Diode:1N4007
- removed J4: Screw_Terminal_01x03, symbol Connector:Screw_Terminal_01x03
- removed J5, J6: Screw_Terminal_01x02, symbol Connector:Screw_Terminal_01x02
- removed JP2, JP3, JP4: Jumper_2_Open, symbol Jumper:Jumper_2_Open
- removed K3: DIPxx-1Cxx-51x, Relay_THT:Relay_StandexMeder_DIP_LowProfile, symbol Relay:DIPxx-1Cxx-51x
- removed Q1, Q3: BC548, Package_TO_SOT_THT:TO-92_Inline, symbol Transistor_BJT:BC548
- removed R11, R3, R4, R5, R8: R, symbol Device:R
- removed U3: PCF8574, symbol Interface_Expansion:PCF8574
- removed U6: PC817, Package_DIP:DIP-4_W7.62mm, symbol Isolator:PC817
- added J4: TRIAC, symbol Connector:Screw_Terminal_01x02
- added Q?: 2N3904, Package_TO_SOT_THT:TO-92_Inline, symbol Transistor_BJT:2N3904
- D11: value LED -> LED TRIAC
- D8: value LED -> LED RELE1
- D9: value LED -> LED RELE2
- J2: value Screw_Terminal_01x03 -> RELE1
- J3: value Screw_Terminal_01x03 -> RELE2
- R6: value R -> 45
- R9: value R -> 5K6
Connections:
- net labels added: COM_RELE1, COM_RELE2, COM_TRIAC, RELE1, RELE1_NA, RELE1_NC, RELE2, RELE2_NA, RELE2_NC, RELE_SS, TRIAC
- net labels removed: 5V, A0, A1, A2, Rele1, Rele2, Rele3, Rele_SS_1, SCL, SDA
- wire segments 105 -> 55
- no-connect marks 5 -> 0
Other:
- note added: "SALIDAS_POTENCIA"
- moved on the sheet: D11, J2, Q4, R13, U7
