File: PLC_ESP32/Alimentacion.sch (KiCad schematic (older format))
At the start: 7 parts, among them J6 Entrada_24VDC, U12 LM7805_TO220, U13 LM7810_TO220

Commit message: -
Parts:
- added D25: BAT760-7 30V 1A, Diode_THT:D_DO-41_SOD81_P10.16mm_Horizontal, symbol Device:D_Schottky
Connections:
- net +5V: now also D25.1 (K); no longer C11.1, D18.2 (A), U12.3 (VO)
- new net: C11.1, D18.2 (A), D25.2 (A), U12.3 (VO)
Changed lines of the file:
@@
 L power:+5V #PWR049
 U 1 1 6146F29E
-P 7200 3150
-F 0 "#PWR049" H 7200 3000 50  0001 C CNN
-F 1 "+5V" H 7215 3323 50  0000 C CNN
-F 2 "" H 7200 3150 50  0001 C CNN
-F 3 "" H 7200 3150 50  0001 C CNN
-	1    7200 3150
+P 7600 3150
+F 0 "#PWR049" H 7600 3000 50  0001 C CNN
+F 1 "+5V" H 7615 3323 50  0000 C CNN
+F 2 "" H 7600 3150 50  0001 C CNN
+F 3 "" H 7600 3150 50  0001 C CNN
+	1    7600 3150
 	1    0    0    -1
 $EndComp
 Wire Wire Line
-	7200 3150 7200 3200
-Wire Wire Line
-	7200 3200 6900 3200
+	7600 3150 7600 3200
 Connection ~ 6900 3200
 $Comp
@@
 Wire Wire Line
 	6000 3200 6100 3200
+$Comp
+L Device:D_Schottky D?
+U 1 1 61F29AFF
+P 7250 3200
+AR Path="/61294432/61F29AFF" Ref="D?"  Part="1"
+AR Path="/612945C2/61F29AFF" Ref="D25"  Part="1"
+F 0 "D25" H 7250 2984 50  0000 C CNN
+F 1 "BAT760-7 30V 1A" H 7250 3075 50  0000 C CNN
+F 2 "Diode_THT:D_DO-41_SOD81_P10.16mm_Horizontal" H 7250 3200 50  0001 C CNN
+F 3 "~" H 7250 3200 50  0001 C CNN
+	1    7250 3200
+	-1   0    0    1
+$EndComp
+Wire Wire Line
+	7100 3200 6900 3200
+Wire Wire Line
+	7400 3200 7600 3200
 $EndSCHEMATC

Commit message: Cambios
Parts:
- D17, D18: footprint Diode_THT:D_DO-41_SOD81_P10.16mm_Horizontal -> Diode_SMD:D_SMA
- U12, U13: footprint Package_TO_SOT_THT:TO-220-3_Vertical -> Package_TO_SOT_THT:TO-220-3_Horizontal_TabUp
Changed lines of the file:
@@
 EESchema Schematic File Version 4
+LIBS:PLC_ESP32-cache
 EELAYER 30 0
 EELAYER END
@@
 F 0 "U12" H 6400 3442 50  0000 C CNN
 F 1 "LM7805_TO220" H 6400 3351 50  0000 C CNN
-F 2 "Package_TO_SOT_THT:TO-220-3_Vertical" H 6400 3425 50  0001 C CIN
+F 2 "Package_TO_SOT_THT:TO-220-3_Horizontal_TabUp" H 6400 3425 50  0001 C CIN
 F 3 "http://www.fairchildsemi.com/ds/LM/LM7805.pdf" H 6400 3150 50  0001 C CNN
 	1    6400 3200
@@
 F 0 "D17" H 5650 2984 50  0000 C CNN
 F 1 "1N4007" H 5650 3075 50  0000 C CNN
-F 2 "Diode_THT:D_DO-41_SOD81_P10.16mm_Horizontal" H 5650 3025 50  0001 C CNN
+F 2 "Diode_SMD:D_SMA" H 5650 3025 50  0001 C CNN
 F 3 "http://www.vishay.com/docs/88503/1n4001.pdf" H 5650 3200 50  0001 C CNN
 	1    5650 3200
@@
 F 0 "U13" H 6400 4442 50  0000 C CNN
 F 1 "LM7810_TO220" H 6400 4351 50  0000 C CNN
-F 2 "Package_TO_SOT_THT:TO-220-3_Vertical" H 6400 4425 50  0001 C CIN
+F 2 "Package_TO_SOT_THT:TO-220-3_Horizontal_TabUp" H 6400 4425 50  0001 C CIN
 F 3 "http://www.fairchildsemi.com/ds/LM/LM7805.pdf" H 6400 4150 50  0001 C CNN
 	1    6400 4200
@@
 F 0 "D18" H 6400 3066 50  0000 C CNN
 F 1 "1N4007" H 6400 2975 50  0000 C CNN
-F 2 "Diode_THT:D_DO-41_SOD81_P10.16mm_Horizontal" H 6400 2675 50  0001 C CNN
+F 2 "Diode_SMD:D_SMA" H 6400 2675 50  0001 C CNN
 F 3 "http://www.vishay.com/docs/88503/1n4001.pdf" H 6400 2850 50  0001 C CNN
 	1    6400 2850
