File: PLC_ESP32/Control.sch (KiCad schematic (older format))
At the start: 36 parts, among them J1 USB_B_Micro, J11 Salida PWM, J12 UART_SERIE, Q1 SS8050-G, Q2 SS8050-G, SW1 SW_Push, SW2 SW_Push, U1 AMS1117-3.3, U2 CP2102N-A01-GQFN28, U3 ESP32-WROOM-32

Commit message: -
Parts:
- removed D2, D3, D4: LESD5D5.0CT1G, symbol Device:D_TVS_ALT
- added JP3: IO2, Connector_PinHeader_2.54mm:PinHeader_1x03_P2.54mm_Vertical, symbol Jumper:Jumper_3_Bridged12
- added JP4, JP6: IO13, Connector_PinHeader_2.54mm:PinHeader_1x03_P2.54mm_Vertical, symbol Jumper:Jumper_3_Bridged12
- added JP5: IO5, Connector_PinHeader_2.54mm:PinHeader_1x03_P2.54mm_Vertical, symbol Jumper:Jumper_3_Bridged12
- added JP7: IO34, Connector_PinHeader_2.54mm:PinHeader_1x02_P2.54mm_Vertical, symbol Device:Jumper
- added R29, R34, R39, R40: 10K(5%), Resistor_SMD:R_0805_2012Metric, symbol Device:R
- added SW3: Rotary_Encoder_Switch, Rotary_Encoder:RotaryEncoder_Alps_EC12E-Switch_Vertical_H20mm, symbol Device:Rotary_Encoder_Switch
- J12: footprint Connector_PinSocket_2.54mm:PinSocket_1x04_P2.54mm_Vertical -> Connector_PinSocket_2.54mm:PinSocket_1x04_P2.54mm_Horizontal
Connections:
- net +3V3: now also R29.2, R34.2, R40.2, SW3.S1
- net A0.0: now also JP6.2 (C); no longer U3.14 (IO12)
- net A0.1: now also U3.7 (IO35); no longer U3.13 (IO14)
- net GND: now also JP3.1 (A), R39.2, SW3.C
- net I0.0: now also U3.14 (IO12); no longer U3.23 (IO15)
- net I0.1: now also U3.13 (IO14); no longer U3.27 (IO16)
- net I0.2: now also U3.23 (IO15); no longer U3.31 (IO19)
- net I0.3: now also U3.27 (IO16); no longer U3.26 (IO4)
- net IO0: now also R40.1
- net IO13: now also JP4.2 (C); no longer J11.1 (Pin_1)
- net IO2: now also JP3.2 (C); no longer BZ1.1 (-)
- net IO5: now also JP5.2 (C); no longer J11.2 (Pin_2)
- net Q0.6: now also U3.31 (IO19); no longer U3.6 (IO34)
- net Q0.7: now also U3.26 (IO4); no longer U3.7 (IO35)
- net SENSOR_VP: now also JP6.3 (B)
- new net: BZ1.1 (-), JP3.3 (B)
- new net: JP7.1, R39.1, SW3.S2
- new net A_ENCODER: JP4.1 (A), R29.1, SW3.A
- new net B_ENCODER: JP5.1 (A), R34.1, SW3.B
- new net IO13_PWM: J11.1 (Pin_1), JP4.3 (B)
- new net IO34: JP6.1 (A), JP7.2, U3.6 (IO34)
- new net IO5_PWM: J11.2 (Pin_2), JP5.3 (B)
- no-connect marks 24 -> 23
Other:
- note added: "1N4937\n1n5819"
- note added: "4.7k"
- note added: "470 ohm\n1K"
- note removed: "1N4937"
- moved on the sheet: BZ1, C8, C9, J11, J12, SW1, SW2

Commit message: Cambios
Parts:
- removed J11: Salida PWM, BorneraTornillos:TerminalBlock_Phoenix_PT-1,5-3-5.0-H_1x03_P5.00mm_Horizontal, symbol Connector:Screw_Terminal_01x03
- removed JP4, JP6: IO13, Connector_PinHeader_2.54mm:PinHeader_1x03_P2.54mm_Vertical, symbol Jumper:Jumper_3_Bridged12
- removed JP5: IO5, Connector_PinHeader_2.54mm:PinHeader_1x03_P2.54mm_Vertical, symbol Jumper:Jumper_3_Bridged12
- removed JP7: IO34, Connector_PinHeader_2.54mm:PinHeader_1x02_P2.54mm_Vertical, symbol Device:Jumper
- removed SW3: Rotary_Encoder_Switch, Rotary_Encoder:RotaryEncoder_Alps_EC12E-Switch_Vertical_H20mm, symbol Device:Rotary_Encoder_Switch
- added D2: LED_RGBC, LED_THT:LED_D5.0mm-4_RGB, symbol Device:LED_RGBC
- R29, R34, R39: value 10K(5%) -> 100 Ohm 1/8W 5%
Connections:
- net IO34 is gone; now on net I0.3: U3.6 (IO34)
- net IO5 is gone; now on net I0.0: U3.29 (IO5)
- net SENSOR_VP is gone; now on net A0.0: U3.4 (SENSOR_VP)
- net +3V3: no longer R29.2, R34.2
- net GND: now also D2.4 (K); no longer R39.2
- net I0.0: no longer U3.14 (IO12)
- net I0.1: now also U3.23 (IO15); no longer U3.13 (IO14)
- net I0.2: now also U3.27 (IO16); no longer U3.23 (IO15)
- net I0.3: no longer U3.27 (IO16)
- net IO13: now also R34.2
- net Q0.0: now also U3.26 (IO4); no longer U3.28 (IO17)
- net Q0.1: now also U3.28 (IO17); no longer U3.30 (IO18)
- net Q0.2: now also U3.30 (IO18); no longer U3.37 (IO23)
- net Q0.3: now also U3.31 (IO19); no longer U3.12 (IO27)
- net Q0.4: now also U3.37 (IO23); no longer U3.8 (IO32)
- net Q0.5: now also U3.12 (IO27); no longer U3.9 (IO33)
- net Q0.6: now also U3.8 (IO32); no longer U3.31 (IO19)
- net Q0.7: now also U3.9 (IO33); no longer U3.26 (IO4)
- net at R39.1: now also D2.1 (RA)
- net A_ENCODER: no longer names the net of R29.1
- net A_ENCODER: now also D2.3 (BA)
- net B_ENCODER: no longer names the net of R34.1
- net B_ENCODER: now also D2.2 (GA)
- new net IO12: R29.2, U3.14 (IO12)
- new net IO14: R39.2, U3.13 (IO14)
Other:
- moved on the sheet: C8, C9, R40, R6, R7, SW1, SW2
