File: PLC_ESP32/Entradas.sch (KiCad schematic (older format))
At the start: 28 parts, among them J13 Entrada Digital, J14 Entrada Digital, J15 Entrada Digital, J16 Entrada Analogica, U14 PC817, U15 LM358, U16 PC817, U17 PC817, U18 PC817

Commit message: Cambios
Parts:
- C12, C13, C14, C15: footprint Capacitor_THT:C_Disc_D5.0mm_W2.5mm_P2.50mm -> Capacitor_SMD:C_0805_2012Metric
Changed lines of the file:
@@
 EESchema Schematic File Version 4
+LIBS:PLC_ESP32-cache
 EELAYER 30 0
 EELAYER END
@@
 F 0 "C12" H 2415 2146 50  0000 L CNN
 F 1 "100nf" H 2415 2055 50  0000 L CNN
-F 2 "Capacitor_THT:C_Disc_D5.0mm_W2.5mm_P2.50mm" H 2338 1950 50  0001 C CNN
+F 2 "Capacitor_SMD:C_0805_2012Metric" H 2338 1950 50  0001 C CNN
 F 3 "~" H 2300 2100 50  0001 C CNN
 	1    2300 2100
@@
 F 0 "C13" H 3865 2146 50  0000 L CNN
 F 1 "100nf" H 3865 2055 50  0000 L CNN
-F 2 "Capacitor_THT:C_Disc_D5.0mm_W2.5mm_P2.50mm" H 3788 1950 50  0001 C CNN
+F 2 "Capacitor_SMD:C_0805_2012Metric" H 3788 1950 50  0001 C CNN
 F 3 "~" H 3750 2100 50  0001 C CNN
 	1    3750 2100
@@
 F 0 "C14" H 5315 2146 50  0000 L CNN
 F 1 "100nf" H 5315 2055 50  0000 L CNN
-F 2 "Capacitor_THT:C_Disc_D5.0mm_W2.5mm_P2.50mm" H 5238 1950 50  0001 C CNN
+F 2 "Capacitor_SMD:C_0805_2012Metric" H 5238 1950 50  0001 C CNN
 F 3 "~" H 5200 2100 50  0001 C CNN
 	1    5200 2100
@@
 F 0 "C15" H 6765 2146 50  0000 L CNN
 F 1 "100nf" H 6765 2055 50  0000 L CNN
-F 2 "Capacitor_THT:C_Disc_D5.0mm_W2.5mm_P2.50mm" H 6688 1950 50  0001 C CNN
+F 2 "Capacitor_SMD:C_0805_2012Metric" H 6688 1950 50  0001 C CNN
 F 3 "~" H 6650 2100 50  0001 C CNN
 	1    6650 2100
