File: PLC_ESP32/Periféricos.sch (KiCad schematic (older format))
At the start: 6 parts, among them J10 Salidas Analogicas, J7 PANTALLA LCD I2C, J8 DS3231, J9 PANTALLA OLED

Commit message: Cambios
Parts:
- removed J8: DS3231, BorneraTornillos:DS3231_Shield, symbol Connector:Conn_01x10_Female
- added A0, A1, A2: Jumper, Jumper:SolderJumper-2_P1.3mm_Open_Pad1.0x1.5mm, symbol Device:Jumper
- added BT1: Battery_Cell, BorneraTornillos:BatteryHolder_Keystone_103_1x20mm, symbol Device:Battery_Cell
- added C16, C17: 0.1uf, Capacitor_SMD:C_0805_2012Metric, symbol Device:C
- added D3: 1N4148, Diode_SMD:D_MELF, symbol Diode:1N4148
- added R41, R42, R43, R45, R46: 4K7 1/8W 5%, Resistor_SMD:R_0805_2012Metric, symbol Device:R
- added R44: 200 1/8W 5%, Resistor_SMD:R_0805_2012Metric, symbol Device:R
- added U19: AT24CS32-XHM, Package_SO:TSSOP-8_4.4x3mm_P0.65mm, symbol Memory_EEPROM:AT24CS32-XHM
- added U20: DS3231M, Package_SO:SOIC-16W_7.5x10.3mm_P1.27mm, symbol Timer_RTC:DS3231M
Connections:
- net +3V3: now also C16.1, C17.1, R41.1, R42.1, R43.1, R44.2, R45.1, R46.1, U19.8 (VCC), U20.2 (VCC)
- net GND: now also A0.1, A1.1, A2.1, BT1.2 (-), C16.2, C17.2, U19.4 (GND), U19.7 (WP), U20.10 (GND), U20.11 (GND), U20.12 (GND), U20.13 (GND), U20.5 (GND), U20.6 (GND), U20.7 (GND), U20.8 (GND), U20.9 (GND)
- net SCL: now also U19.6 (SCL), U20.16 (SCL)
- net SDA: now also U19.5 (SDA), U20.15 (SDA)
- new net: R45.2, U20.1 (32KHZ)
- new net: BT1.1 (+), D3.1 (K), U20.14 (VBAT)
- new net: R46.2, U20.3 (~INT~/SQW)
- new net: D3.2 (A), R44.1
- new net: A0.2, R43.2, U19.1 (A0)
- new net: A1.2, R42.2, U19.2 (A1)
- new net: A2.2, R41.2, U19.3 (A2)
- no-connect marks 6 -> 1
Other:
- note added: "RTC y EEPROM"
- moved on the sheet: J10, J7, J9, R37, R38
