File: PLC_ESP32/Salidas.sch (KiCad schematic (older format))
At the start: 50 parts, among them J2 Terminales Reles, J3 Terminales Reles, J4 Terminales Triacs, J5 Terminales Triacs, K1 SANYOU_SRD_Form_C, K2 SANYOU_SRD_Form_C, K3 SANYOU_SRD_Form_C, Q10 BT136-500, Q3 2N2222A, Q4 2N2222A, Q5 2N2222A, Q6 BT136-500, Q7 BT136-500, Q8 BT136-500, Q9 BT136-500, U10 MOC3021M, U11 MOC3021M, U4 PC817, U5 PC817, U6 PC817, U7 MOC3021M, U8 MOC3021M, U9 MOC3021M

Commit message: -
Changed lines of the file:
@@
 Text Notes 1400 850  0    50   ~ 0
 Rrele= 70 ohm
+$Comp
+L power:PWR_FLAG #FLG0104
+U 1 1 62398517
+P 2400 800
+F 0 "#FLG0104" H 2400 875 50  0001 C CNN
+F 1 "PWR_FLAG" H 2400 973 50  0000 C CNN
+F 2 "" H 2400 800 50  0001 C CNN
+F 3 "~" H 2400 800 50  0001 C CNN
+	1    2400 800
+	1    0    0    -1
+$EndComp
+Wire Wire Line
+	2400 800  2400 900
+Wire Wire Line
+	2400 900  2100 900
 $EndSCHEMATC

Commit message: Cambios
Parts:
- removed Q3, Q4, Q5: 2N2222A, Package_TO_SOT_THT:TO-92_Inline, symbol Transistor_BJT:BC548
- added Q3, Q4, Q5: 2N2219, Package_TO_SOT_THT:TO-92_Inline, symbol Transistor_BJT:2N2219
- D11, D8, D9: footprint Diode_THT:D_DO-41_SOD81_P10.16mm_Horizontal -> Diode_SMD:D_SMA
Connections:
- net GND: now also Q3.1 (E), Q4.1 (E), Q5.1 (E)
- net at D8.2 (A), K1.2: now also Q3.3 (C)
- net at R13.2: now also Q3.2 (B)
- net at D9.2 (A), K2.2: now also Q4.3 (C)
- net at R14.2: now also Q4.2 (B)
- net at D11.2 (A), K3.2: now also Q5.3 (C)
- net at R16.2: now also Q5.2 (B)
Changed lines of the file:
@@
 EESchema Schematic File Version 4
+LIBS:PLC_ESP32-cache
 EELAYER 30 0
 EELAYER END
@@
 $EndComp
 $Comp
-L Transistor_BJT:BC548 Q3
-U 1 1 6145D2A0
-P 2000 1900
-AR Path="/61294493/6145D2A0" Ref="Q3"  Part="1"
-AR Path="/615E1DF0/6145D2A0" Ref="Q?"  Part="1"
-F 0 "Q3" H 2191 1946 50  0000 L CNN
-F 1 "2N2222A" H 2191 1855 50  0000 L CNN
-F 2 "Package_TO_SOT_THT:TO-92_Inline" H 2200 1825 50  0001 L CIN
-F 3 "http://www.fairchildsemi.com/ds/BC/BC547.pdf" H 2000 1900 50  0001 L CNN
-	1    2000 1900
-	1    0    0    -1
-$EndComp
-$Comp
 L Device:R R13
 U 1 1 6145E3DC
@@
 F 0 "D8" V 1650 1300 50  0000 L CNN
 F 1 "1N4007" H 1600 1100 50  0000 L CNN
-F 2 "Diode_THT:D_DO-41_SOD81_P10.16mm_Horizontal" H 1750 1075 50  0001 C CNN
+F 2 "Diode_SMD:D_SMA" H 1750 1075 50  0001 C CNN
 F 3 "http://www.vishay.com/docs/88503/1n4001.pdf" H 1750 1250 50  0001 C CNN
 	1    1750 1250
@@
 $EndComp
 $Comp
-L Transistor_BJT:BC548 Q4
-U 1 1 6147F0A4
-P 2100 4200
-AR Path="/61294493/6147F0A4" Ref="Q4"  Part="1"
-AR Path="/615E1DF0/6147F0A4" Ref="Q?"  Part="1"
-F 0 "Q4" H 2291 4246 50  0000 L CNN
-F 1 "2N2222A" H 2291 4155 50  0000 L CNN
-F 2 "Package_TO_SOT_THT:TO-92_Inline" H 2300 4125 50  0001 L CIN
-F 3 "http://www.fairchildsemi.com/ds/BC/BC547.pdf" H 2100 4200 50  0001 L CNN
-	1    2100 4200
-	1    0    0    -1
-$EndComp
-$Comp
 L Device:R R14
 U 1 1 6147F0AE
@@
 F 0 "D9" V 1750 3600 50  0000 L CNN
 F 1 "1N4007" H 1700 3400 50  0000 L CNN
-F 2 "Diode_THT:D_DO-41_SOD81_P10.16mm_Horizontal" H 1850 3375 50  0001 C CNN
+F 2 "Diode_SMD:D_SMA" H 1850 3375 50  0001 C CNN
 F 3 "http://www.vishay.com/docs/88503/1n4001.pdf" H 1850 3550 50  0001 C CNN
 	1    1850 3550
@@
 $EndComp
 $Comp
-L Transistor_BJT:BC548 Q5
-U 1 1 6148BC50
-P 4450 1900
-AR Path="/61294493/6148BC50" Ref="Q5"  Part="1"
-AR Path="/615E1DF0/6148BC50" Ref="Q?"  Part="1"
-F 0 "Q5" H 4641 1946 50  0000 L CNN
-F 1 "2N2222A" H 4641 1855 50  0000 L CNN
-F 2 "Package_TO_SOT_THT:TO-92_Inline" H 4650 1825 50  0001 L CIN
-F 3 "http://www.fairchildsemi.com/ds/BC/BC547.pdf" H 4450 1900 50  0001 L CNN
-	1    4450 1900
-	1    0    0    -1
-$EndComp
-$Comp
 L Device:R R16
 U 1 1 6148BC5A
@@
 F 0 "D11" V 4100 1300 50  0000 L CNN
 F 1 "1N4007" H 4050 1100 50  0000 L CNN
-F 2 "Diode_THT:D_DO-41_SOD81_P10.16mm_Horizontal" H 4200 1075 50  0001 C CNN
+F 2 "Diode_SMD:D_SMA" H 4200 1075 50  0001 C CNN
 F 3 "http://www.vishay.com/docs/88503/1n4001.pdf" H 4200 1250 50  0001 C CNN
 	1    4200 1250
@@
 Wire Wire Line
 	2400 900  2100 900
+$Comp
+L Transistor_BJT:2N2219 Q3
+U 1 1 6154F61B
+P 2000 1900
+F 0 "Q3" H 2190 1946 50  0000 L CNN
+F 1 "2N2219" H 2190 1855 50  0000 L CNN
+F 2 "Package_TO_SOT_THT:TO-92_Inline" H 2200 1825 50  0001 L CIN
+F 3 "http://www.onsemi.com/pub_link/Collateral/2N2219-D.PDF" H 2000 1900 50  0001 L CNN
+	1    2000 1900
+	1    0    0    -1
+$EndComp
+$Comp
+L Transistor_BJT:2N2219 Q5
+U 1 1 61550A00
+P 4450 1900
+F 0 "Q5" H 4640 1946 50  0000 L CNN
+F 1 "2N2219" H 4640 1855 50  0000 L CNN
+F 2 "Package_TO_SOT_THT:TO-92_Inline" H 4650 1825 50  0001 L CIN
+F 3 "http://www.onsemi.com/pub_link/Collateral/2N2219-D.PDF" H 4450 1900 50  0001 L CNN
+	1    4450 1900
+	1    0    0    -1
+$EndComp
+$Comp
+L Transistor_BJT:2N2219 Q4
+U 1 1 6155197A
+P 2100 4200
+F 0 "Q4" H 2290 4246 50  0000 L CNN
+F 1 "2N2219" H 2290 4155 50  0000 L CNN
+F 2 "Package_TO_SOT_THT:TO-92_Inline" H 2300 4125 50  0001 L CIN
+F 3 "http://www.onsemi.com/pub_link/Collateral/2N2219-D.PDF" H 2100 4200 50  0001 L CNN
+	1    2100 4200
+	1    0    0    -1
+$EndComp
 $EndSCHEMATC
