File: PLC_ESP32/PLC_ESP32.kicad_pcb (KiCad board)
At the start: 2 copper layers, 100 x 100 mm, 128 parts, among them J1 USB_B_Micro, J10 Salidas Analogicas, J11 Salida PWM, J12 UART_SERIE, J13 Entrada Digital, J14 Entrada Digital, J15 Entrada Digital, J16 Entrada Analogica, J2 Terminales Reles, J3 Terminales Reles, J4 Terminales Triacs, J5 Terminales Triacs, J6 Entrada_24VDC, J7 PANTALLA LCD I2C, J8 DS3231, J9 PANTALLA OLED, K1 SANYOU_SRD_Form_C, K2 SANYOU_SRD_Form_C, K3 SANYOU_SRD_Form_C, Q1 SS8050-G, Q10 BT136-500, Q2 SS8050-G, Q3 2N2222A, Q4 2N2222A, Q5 2N2222A, Q6 BT136-500, Q7 BT136-500, Q8 BT136-500, Q9 BT136-500, SW1 SW_Push, SW2 SW_Push, U1 AMS1117-3.3, U10 MOC3021M, U11 MOC3021M, U12 LM7805_TO220, U13 LM7810_TO220, U14 PC817, U15 LM358, U16 PC817, U17 PC817, U18 PC817, U2 CP2102N-A01-GQFN28, U3 ESP32-WROOM-32, U4 PC817, U5 PC817, U6 PC817, U7 MOC3021M, U8 MOC3021M, U9 MOC3021M

Commit message: -
Parts:
- added D25: BAT760-7 30V 1A, Diode_THT:D_DO-41_SOD81_P10.16mm_Horizontal, F.Cu at (116.1, 137.3)
- added JP3: IO2, Connector_PinHeader_2.54mm:PinHeader_1x03_P2.54mm_Vertical, F.Cu at (145.9, 109.4)
- added JP4: IO13, Connector_PinHeader_2.54mm:PinHeader_1x03_P2.54mm_Vertical, F.Cu at (145.9, 115.2)
- added JP5: IO5, Connector_PinHeader_2.54mm:PinHeader_1x03_P2.54mm_Vertical, F.Cu at (155.1, 109.4)
- added JP6: IO13, Connector_PinHeader_2.54mm:PinHeader_1x03_P2.54mm_Vertical, F.Cu at (155.1, 115.2)
- added JP7: IO34, Connector_PinHeader_2.54mm:PinHeader_1x02_P2.54mm_Vertical, F.Cu at (168.5, 157.4)
- added R29: 10K(5%), Resistor_SMD:R_0805_2012Metric, F.Cu at (152.8, 130.9)
- added R34: 10K(5%), Resistor_SMD:R_0805_2012Metric, F.Cu at (152.8, 133.1)
- added R39: 10K(5%), Resistor_SMD:R_0805_2012Metric, F.Cu at (156.5, 130.9)
- added R40: 10K(5%), Resistor_SMD:R_0805_2012Metric, F.Cu at (156.5, 133.1)
- added REF5: KiCad-Logo2_20mm_SilkScreen, Symbol:KiCad-Logo2_20mm_SilkScreen, B.Cu at (112.3, 127.2)
- added SW3: Rotary_Encoder_Switch, Rotary_Encoder:RotaryEncoder_Alps_EC12E-Switch_Vertical_H20mm, F.Cu at (156.5, 163.3)
- J12: footprint Connector_PinSocket_2.54mm:PinSocket_1x04_P2.54mm_Vertical -> Connector_PinSocket_2.54mm:PinSocket_1x04_P2.54mm_Horizontal; moved to B.Cu
- J7: moved to B.Cu
- moved J12 43.7 mm to (92.6, 118.5), turned to 0 degrees
- moved C5 32.7 mm to (100.2, 116.9), turned to 90 degrees
- moved C9 30.5 mm to (102.3, 116.8), turned to 270 degrees
- moved BZ1 21.1 mm to (173.2, 114.3), turned to 90 degrees
- moved R11 20.5 mm to (105.6, 133.3), turned to 90 degrees
- moved C3 19.1 mm to (107.8, 133.3), turned to 90 degrees
- moved D23 13.1 mm to (163.7, 139.0), turned to 90 degrees
- moved J15 11.3 mm to (131.9, 157.2)
- moved J16 11.3 mm to (142.4, 157.2)
- moved J13 11.3 mm to (101.0, 157.2)
- moved J14 11.3 mm to (116.5, 157.2)
- moved D1 10.7 mm to (109.5, 118.2)
- moved C15 10.6 mm to (160.3, 144.6)
- moved C6 10.5 mm to (109.5, 116.0)
- moved JP2 9.99 mm to (173.5, 152.1)
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Connections:
- BZ1 pad 1: /Control/IO2 -> Net-(BZ1-Pad1)
- C11 pad 1: +5V -> Net-(C11-Pad1)
- D18 pad 2: +5V -> Net-(C11-Pad1)
- J11 pad 1: /Control/IO13 -> /Control/IO13_PWM
- J11 pad 2: /Control/IO5 -> /Control/IO5_PWM
- U12 pad 3: +5V -> Net-(C11-Pad1)
- U3 pad 13: /Control/A0.1 -> /Control/I0.1
- U3 pad 14: /Control/A0.0 -> /Control/I0.0
- U3 pad 23: /Control/I0.0 -> /Control/I0.2
- U3 pad 26: /Control/I0.3 -> /Control/Q0.7
- U3 pad 27: /Control/I0.1 -> /Control/I0.3
- U3 pad 31: /Control/I0.2 -> /Control/Q0.6
- U3 pad 6: /Control/Q0.6 -> /Control/IO34
- U3 pad 7: /Control/Q0.7 -> /Control/A0.1
Routing:
- net /Control/B_ENCODER: track 0.00 -> 123.9 mm, vias 0 -> 1
- net /Control/IO34: track 0.00 -> 92.3 mm, vias 0 -> 2
- net +3V3: track 282.8 -> 372.5 mm
- net /Control/A_ENCODER: track 0.00 -> 78.7 mm, vias 0 -> 2
- net /Control/EN: track 97.4 -> 170.5 mm, vias 2 -> 3
- net /Control/IO0: track 54.8 -> 118.0 mm, vias 1 -> 3
- net /Control/A0.0: track 63.7 -> 111.9 mm, vias 2 -> 0
- net /Control/IO13: track 86.7 -> 41.3 mm, vias 0 -> 1
- net /Control/SENSOR_VP: track 0.00 -> 39.3 mm, vias 0 -> 2
- net /Control/SCL: track 112.9 -> 74.3 mm, vias 1 -> 3
- net /Control/Q0.6: track 56.0 -> 92.0 mm
- net /Control/RXD0: track 67.7 -> 103.3 mm, vias 2 -> 3
- net Net-(JP7-Pad1): track 0.00 -> 35.1 mm, vias 0 -> 3
- net Net-(C11-Pad1): track 0.00 -> 34.3 mm
- net Net-(D22-Pad2): track 112.2 -> 79.6 mm
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- added copper zone on B.Cu, net GND
- added copper zone on F.Cu, net GND
Other:
- outline, holes or cut-outs redrawn
- net class Alimentacion added: clearance 0.2, trace_width 0.5, via_dia 0.8, via_drill 0.4
- rule trace_min: 0.2 -> 0.25
- board text added: "DAC0.0 DAC0.1 GND"
- board text added: "ENC|IO13|PWM"
- board text added: "ENC|IO5|PWM"
- board text added: "GND|I02|BUZ"
- board text added: "I034"
- board text added: "I034|A0.0|SENVP"
- board text added: "IO0"
- board text added: "PLC ESP32 V1.0 Agustin Zuliani"
- board text added: "PWM1 PWM2 GND"
- board text removed: "EN"

Commit message: Cambios
Parts:
- removed J11: Salida PWM, BorneraTornillos:TerminalBlock_Phoenix_PT-1,5-3-5.0-H_1x03_P5.00mm_Horizontal
- removed J8: DS3231, BorneraTornillos:DS3231_Shield
- removed JP4, JP6: IO13, Connector_PinHeader_2.54mm:PinHeader_1x03_P2.54mm_Vertical
- removed JP5: IO5, Connector_PinHeader_2.54mm:PinHeader_1x03_P2.54mm_Vertical
- removed JP7: IO34, Connector_PinHeader_2.54mm:PinHeader_1x02_P2.54mm_Vertical
- removed REF1, REF2, REF3, REF4: MountingHole_3.2mm_M3_Pad, MountingHole:MountingHole_3.2mm_M3_Pad
- removed REF5: KiCad-Logo2_20mm_SilkScreen, Symbol:KiCad-Logo2_20mm_SilkScreen
- removed SW3: Rotary_Encoder_Switch, Rotary_Encoder:RotaryEncoder_Alps_EC12E-Switch_Vertical_H20mm
- added A0: Jumper, Jumper:SolderJumper-2_P1.3mm_Open_Pad1.0x1.5mm, F.Cu at (162.0, 135.0)
- added A1: Jumper, Jumper:SolderJumper-2_P1.3mm_Open_Pad1.0x1.5mm, F.Cu at (164.5, 135.0)
- added A2: Jumper, Jumper:SolderJumper-2_P1.3mm_Open_Pad1.0x1.5mm, F.Cu at (167.0, 135.0)
- added BT1: Battery_Cell, BorneraTornillos:BatteryHolder_Keystone_103_1x20mm, B.Cu at (149.0, 142.5)
- added C16: 0.1uf, Capacitor_SMD:C_0805_2012Metric, B.Cu at (174.0, 111.5)
- added C17: 0.1uf, Capacitor_SMD:C_0805_2012Metric, B.Cu at (174.0, 114.0)
- added D2: LED_RGBC, LED_THT:LED_D5.0mm-4_RGB, F.Cu at (111.5, 117.0)
- added D3: 1N4148, Diode_SMD:D_MELF, B.Cu at (141.0, 109.5)
- added R41: 4K7 1/8W 5%, Resistor_SMD:R_0805_2012Metric, B.Cu at (173.5, 123.5)
- added R42: 4K7 1/8W 5%, Resistor_SMD:R_0805_2012Metric, B.Cu at (169.5, 123.5)
- added R43: 4K7 1/8W 5%, Resistor_SMD:R_0805_2012Metric, B.Cu at (165.0, 123.5)
- added R44: 200 1/8W 5%, Resistor_SMD:R_0805_2012Metric, B.Cu at (144.5, 111.0)
- added R45: 4K7 1/8W 5%, Resistor_SMD:R_0805_2012Metric, B.Cu at (174.0, 104.5)
- added R46: 4K7 1/8W 5%, Resistor_SMD:R_0805_2012Metric, B.Cu at (174.0, 107.0)
- added U19: AT24CS32-XHM, Package_SO:TSSOP-8_4.4x3mm_P0.65mm, F.Cu at (171.0, 129.0)
- added U20: DS3231M, Package_SO:SOIC-16W_7.5x10.3mm_P1.27mm, B.Cu at (156.2, 109.8)
- C12, C13, C14, C15: footprint Capacitor_THT:C_Disc_D5.0mm_W2.5mm_P2.50mm -> Capacitor_SMD:C_0805_2012Metric
- C5, C6, C8, C9, R1, R11, R12, R13, R14, R15, R16, R17, R18, R19, R2, R23, R24, R3, R4, R5, R6: moved to B.Cu
- D11, D17, D18, D8, D9: footprint Diode_THT:D_DO-41_SOD81_P10.16mm_Horizontal -> Diode_SMD:D_SMA
- Q3, Q4, Q5: value 2N2222A -> 2N2219
- R29, R34, R39: value 10K(5%) -> 100 Ohm 1/8W 5%; moved to B.Cu
- U12, U13: footprint Package_TO_SOT_THT:TO-220-3_Vertical -> Package_TO_SOT_THT:TO-220-3_Horizontal_TabUp; moved to B.Cu
- moved R36 48.6 mm to (151.5, 150.5)
- moved C15 48.4 mm to (113.0, 134.5)
- moved R40 47.8 mm to (109.0, 138.0)
- moved C14 43.7 mm to (113.0, 131.0)
- moved R4 43.5 mm to (132.5, 127.0), turned to 270 degrees
- moved C12 41.3 mm to (113.0, 124.0)
- moved R3 41.3 mm to (125.0, 132.1), turned to 90 degrees
- moved R5 41.3 mm to (122.3, 132.1), turned to 270 degrees
- moved R39 40.5 mm to (118.5, 117.0)
- moved R2 39.0 mm to (125.0, 127.0)
- moved R34 36.9 mm to (118.5, 119.5)
- moved R33 35.8 mm to (138.5, 150.5)
- moved R29 35.4 mm to (118.5, 122.0)
- moved C7 35.4 mm to (113.0, 138.0)
- moved C13 34.6 mm to (113.0, 127.5)
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Connections:
- Q3 pad 1: Net-(D8-Pad2) -> GND
- Q3 pad 3: GND -> Net-(D8-Pad2)
- Q4 pad 1: Net-(D9-Pad2) -> GND
- Q4 pad 3: GND -> Net-(D9-Pad2)
- Q5 pad 1: Net-(D11-Pad2) -> GND
- Q5 pad 3: GND -> Net-(D11-Pad2)
- R29 pad 1: /Control/A_ENCODER -> Net-(D2-Pad3)
- R29 pad 2: +3V3 -> /Control/IO12
- R34 pad 1: /Control/B_ENCODER -> Net-(D2-Pad2)
- R34 pad 2: +3V3 -> /Control/IO13
- R39 pad 2: GND -> /Control/IO14
- U3 pad 12: /Control/Q0.3 -> /Control/Q0.5
- U3 pad 13: /Control/I0.1 -> /Control/IO14
- U3 pad 14: /Control/I0.0 -> /Control/IO12
- U3 pad 23: /Control/I0.2 -> /Control/I0.1
- U3 pad 26: /Control/Q0.7 -> /Control/Q0.0
- U3 pad 27: /Control/I0.3 -> /Control/I0.2
- U3 pad 28: /Control/Q0.0 -> /Control/Q0.1
- U3 pad 29: /Control/IO5 -> /Control/I0.0
- U3 pad 30: /Control/Q0.1 -> /Control/Q0.2
- U3 pad 31: /Control/Q0.6 -> /Control/Q0.3
- U3 pad 37: /Control/Q0.2 -> /Control/Q0.4
- U3 pad 4: /Control/SENSOR_VP -> /Control/A0.0
- U3 pad 6: /Control/IO34 -> /Control/I0.3
- U3 pad 8: /Control/Q0.4 -> /Control/Q0.6
- U3 pad 9: /Control/Q0.5 -> /Control/Q0.7
Routing:
- net /Control/B_ENCODER: track 123.9 -> 0.00 mm, vias 1 -> 0
- net /Control/IO34: track 92.3 -> 0.00 mm, vias 2 -> 0
- net +3V3: track 372.5 -> 282.2 mm, vias 5 -> 2
- net /Control/A_ENCODER: track 78.7 -> 0.00 mm, vias 2 -> 0
- net /Control/EN: track 170.5 -> 97.2 mm
- net /Control/A0.0: track 111.9 -> 52.5 mm, vias 0 -> 1
- net /Control/IO5: track 59.0 -> 0.00 mm, vias 1 -> 0
- net /Control/RXD0: track 103.3 -> 56.3 mm, vias 3 -> 2
- net Net-(BT1-Pad1): track 0.00 -> 46.9 mm
- net /Control/Q0.6: track 92.0 -> 49.3 mm, vias 1 -> 0
- net Net-(R36-Pad1): track 49.9 -> 10.3 mm
- net /Control/SENSOR_VP: track 39.3 -> 0.00 mm, vias 2 -> 0
- net /Entradas/AN0.1: track 51.9 -> 12.9 mm
- net /Control/IO13: track 41.3 -> 4.92 mm
- net Net-(D10-Pad2): track 63.4 -> 27.9 mm, vias 0 -> 1
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Other:
- outline, holes or cut-outs redrawn
- net class 3.3V added: clearance 0.2, trace_width 0.3, via_dia 0.8, via_drill 0.4
- board text added: "POWER"
- board text removed: "ENC|IO13|PWM"
- board text removed: "ENC|IO5|PWM"
- board text removed: "I034"
- board text removed: "I034|A0.0|SENVP"
- board text removed: "PWM1 PWM2 GND"

Commit message: Actualizacion PCB
Parts:
- added REF1: MountingHole_3.2mm_M3_Pad_Via, MountingHole:MountingHole_3.2mm_M3_Pad_Via, F.Cu at (84.2, 69.0)
- added REF1: MountingHole_3.2mm_M3_Pad_Via, MountingHole:MountingHole_3.2mm_M3_Pad_Via, F.Cu at (176.2, 69.0)
- added REF1: MountingHole_3.2mm_M3_Pad_Via, MountingHole:MountingHole_3.2mm_M3_Pad_Via, F.Cu at (176.2, 161.0)
- added REF1: MountingHole_3.2mm_M3_Pad_Via, MountingHole:MountingHole_3.2mm_M3_Pad_Via, F.Cu at (83.8, 161.0)
Other:
- outline, holes or cut-outs redrawn
