File: Inyectores_RPI_PICO/P_Inyectores_Rpi_pico/Control.sch (KiCad schematic (older format))
At the start: 72 parts, among them K1 SANYOU_SRD_Form_C, K2 SANYOU_SRD_Form_C, Q1 IRF540N, Q2 IRF540N, Q3 IRF540N, Q4 IRF540N, Q5 BC548, Q6 BC548, Q7 BC548, SW2 Reset_Push, SW3 Rotary_Encoder_Switch, U1 PC817, U10 DS3231M, U11 AT24CS32-XHM, U2 PC817, U3 PC817, U4 PC817, U7 Pico, U8 PC817, U9 PC817

Commit message: Actualizacion PCB
Parts:
- removed Uart1: Screw_Terminal_01x02, Connector_Molex:Molex_KK-254_AE-6410-02A_1x02_P2.54mm_Vertical, symbol Connector:Screw_Terminal_01x02
- added C10, C11, C12, C13, C14, C9: 104, Capacitor_THT:C_Disc_D5.0mm_W2.5mm_P2.50mm, symbol Device:C
- added J2: Conn_01x07_Male, Connector_PinSocket_2.54mm:PinSocket_1x07_P2.54mm_Vertical, symbol Connector:Conn_01x07_Male
- added R25, R26: 10k, Resistor_THT:R_Axial_DIN0207_L6.3mm_D2.5mm_P10.16mm_Horizontal, symbol Device:R
- added SW1: PUSH2, Button_Switch_THT:SW_PUSH_6mm, symbol Switch:SW_Push
- added SW4: PUSH1, Button_Switch_THT:SW_PUSH_6mm, symbol Switch:SW_Push
- added Uart1: Screw_Terminal_01x02, Connector_Molex:Molex_KK-254_AE-6410-04A_1x04_P2.54mm_Vertical, symbol Connector:Screw_Terminal_01x04
- D9: footprint LED_THT:LED_D5.0mm-4_RGB -> LED_THT:LED_D5.0mm-4_RGB_Wide_Pins
- Q5, Q6, Q7: footprint Package_TO_SOT_THT:TO-92_Inline -> Package_TO_SOT_THT:TO-92_Inline_Wide
- R13: value R -> 12k
- R19, R20, R21, R22, R23, R24: footprint Resistor_THT:R_Axial_DIN0207_L6.3mm_D2.5mm_P10.16mm_Horizontal -> Resistor_SMD:R_0805_2012Metric
- R2: value 53k -> 4k7
Connections:
- net +3V3: now also SW1.1, SW4.1
- net +5V: now also C11.1, C12.1, C13.1, C14.1, Uart1.1 (Pin_1)
- net A: now also C9.1
- net B: now also C10.1
- net GND: now also C10.2, C9.2, R25.1, R26.1, Uart1.4 (Pin_4)
- net UART0_RX: now also Uart1.2 (Pin_2)
- net UART0_TX: now also Uart1.3 (Pin_3)
- net GPIO14: now reaches U7.19 (GPIO14)
- net GPIO14: now also J2.1 (Pin_1)
- net GPIO15: now reaches U7.20 (GPIO15)
- net GPIO15: now also J2.2 (Pin_2)
- net GPIO16: now reaches U7.21 (GPIO16)
- net GPIO16: now also J2.3 (Pin_3)
- net GPIO17: now reaches U7.22 (GPIO17)
- net GPIO17: now also J2.4 (Pin_4)
- net PULSADOR_1: now reaches U7.24 (GPIO18)
- net PULSADOR_1: now also R26.2, SW4.2
- net PULSADOR_2: now reaches U7.25 (GPIO19)
- net PULSADOR_2: now also R25.2, SW1.2
- net GPIO20: now reaches U7.26 (GPIO20)
- net GPIO20: now also J2.5 (Pin_5)
- net GPIO21: now reaches U7.27 (GPIO21)
- net GPIO21: now also J2.6 (Pin_6)
- net GPIO22: now reaches U7.29 (GPIO22)
- net GPIO22: now also J2.7 (Pin_7)
- net at C3.1, Q1.1 (G), R11.2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: now also C11.2
- net at C5.1, Q2.1 (G), R16.2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: now also C13.2
- net at C4.1, Q3.1 (G), R12.2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: now also C12.2
- net at C6.1, Q4.1 (G), R17.2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: now also C14.2
- no-connect marks 28 -> 19
Other:
- moved on the sheet: BZ1, D9, Q5, R2, R3, R4, R6, SW2, SW3

Commit message: -
Parts:
- U11: footprint Package_SO:TSSOP-8_4.4x3mm_P0.65mm -> Package_SO:SOIC-8_3.9x4.9mm_P1.27mm
Changed lines of the file:
@@
 F 0 "U11" H 10350 4131 50  0000 C CNN
 F 1 "AT24CS32-XHM" H 10350 4040 50  0000 C CNN
-F 2 "Package_SO:TSSOP-8_4.4x3mm_P0.65mm" H 10350 3650 50  0001 C CNN
+F 2 "Package_SO:SOIC-8_3.9x4.9mm_P1.27mm" H 10350 3650 50  0001 C CNN
 F 3 "http://ww1.microchip.com/downloads/en/DeviceDoc/Atmel-8869-SEEPROM-AT24CS32-Datasheet.pdf" H 10350 3650 50  0001 C CNN
 	1    10350 3650
