File: Fuente de Alimentacion Nueva CSJ/Fte_Alimentacion/Control.kicad_sch (KiCad schematic)
At the start: 0 parts

Commit message: Avance
Parts:
- added BZ1: Buzzer, symbol Device:Buzzer
- added D13: LED_RGBK, symbol Device:LED_RGBK
- added D14, D15: 1N4007, Diode_THT:D_DO-41_SOD81_P10.16mm_Horizontal, symbol Diode:1N4007
- added J5, J6: Screw_Terminal_01x03, symbol Connector:Screw_Terminal_01x03
- added K1, K2: SANYOU_SRD_Form_C, Relay_THT:Relay_SPDT_SANYOU_SRD_Series_Form_C, symbol Relay:SANYOU_SRD_Form_C
- added Q1, Q2: BC548, Package_TO_SOT_THT:TO-92_Inline, symbol Transistor_BJT:BC548
- added R10, R11, R4, R9: R, symbol Device:R
- added R12: R_JUMP1, symbol Device:R
- added R13: R_JUMP2, symbol Device:R
- added R5, R6, R7, R8: 10k, symbol Device:R
- added SW2, SW3, SW4, SW5: SW_Push, symbol Switch:SW_Push
- added U4: Pico, RPi_Pico:RPi_Pico_SMD_TH, symbol MCU_RaspberryPi_and_Boards:Pico
- added U5, U6: PC817, Package_DIP:DIP-4_W7.62mm, symbol Isolator:PC817
Connections:
- new net: R9.2, U6.1
- new net: R4.2, U5.1
- new net: R10.1, U5.3
- new net: Q1.2 (B), R10.2
- new net: R11.1, U6.3
- new net: Q2.2 (B), R11.2
- new net: D14.2 (A), K1.2, Q1.1 (C)
- new net: K2.1, R13.2
- new net: D15.2 (A), K2.2, Q2.1 (C)
- new net: J6.3 (Pin_3), K2.4
- new net: J5.2 (Pin_2), R12.1
- new net: K1.1, R12.2
- new net: J6.2 (Pin_2), R13.1
- new net +3V3: R8.1, SW2.2, SW3.2, SW4.2
- new net +5V: D14.1 (K), D15.1 (K), K1.5, K2.5, U5.4, U6.4
- new net 3V3: U4.36 (3V3)
- new net 3V3_EN: U4.37 (3V3_EN)
- new net GND: BZ1.2 (+), D13.4 (K), Q1.3 (E), Q2.3 (E), R5.2, R6.2, R7.2, SW5.1, U4.3 (GND), U4.33 (AGND), U5.2, U6.2
- new net GPIO0: U4.1 (GPIO0)
- new net GPIO1: U4.2 (GPIO1)
- new net GPIO10: R9.1, U4.14 (GPIO10)
- new net GPIO11: R5.1, SW2.1, U4.15 (GPIO11)
- new net GPIO12: R6.1, SW3.1, U4.16 (GPIO12)
- new net GPIO13: R7.1, SW4.1, U4.17 (GPIO13)
- new net GPIO14: D13.3 (BA), U4.19 (GPIO14)
- new net GPIO15: D13.2 (GA), U4.20 (GPIO15)
- new net GPIO16: D13.1 (RA), U4.21 (GPIO16)
- new net GPIO17: BZ1.1 (-), U4.22 (GPIO17)
- new net GPIO18: U4.24 (GPIO18)
- new net GPIO19: U4.25 (GPIO19)
- new net GPIO2: U4.4 (GPIO2)
- new net GPIO20: U4.26 (GPIO20)
- new net GPIO21: U4.27 (GPIO21)
- new net GPIO22: U4.29 (GPIO22)
- new net GPIO26: U4.31 (GPIO26_ADC0)
- new net GPIO27: U4.32 (GPIO27_ADC1)
- new net GPIO28: U4.34 (GPIO28_ADC2)
- new net GPIO3: U4.5 (GPIO3)
- new net GPIO4: U4.6 (GPIO4)
- new net GPIO5: U4.7 (GPIO5)
- new net GPIO6: U4.9 (GPIO6)
- new net GPIO7: U4.10 (GPIO7)
- new net GPIO8: U4.11 (GPIO8)
- new net GPIO9: R4.1, U4.12 (GPIO9)
- new net RUN: R8.2, SW5.2, U4.30 (RUN)
- no-connect marks 0 -> 12
